File: leds/dashboard_leds.kicad_pcb (KiCad board)
At the start: 4 copper layers, 21 x 76.6 mm, 48 parts, among them J1 Harness, J2 Conn_01x06, J3 Expansion Connector, Q1 BSS138, Q2 BSS138, Q3 BSS138, Q4 BSS138, Q5 BSS138

Commit message: Updating one resistor value on pcb
Parts:
- R20: value 150 -> 100
Changed lines of the file:
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@@
 			)
 		)
-		(property "Value" "150"
+		(property "Value" "100"
 			(at 0 1.82 0)
 			(layer "F.Fab")
